File: RI279C.kicad_pcb (KiCad board)
At the start: 2 copper layers, 49 x 39 mm, 10 parts, among them J1 Ribbon Cable, J2 Multiway, J3 Meter

Commit message: added TAC library as submodule
Parts:
- SK2, SK3: footprint Cliff:CL13345 -> TAC:CL13345
