File: RI279C.sch (KiCad schematic (older format))
At the start: 10 parts, among them J1 Ribbon Cable, J2 Multiway, J3 Meter

Commit message: added TAC library as submodule
Parts:
- SK2, SK3: footprint Cliff:CL13345 -> TAC:CL13345
Changed lines of the file:
@@
 F 0 "SK2" H 2150 2950 50  0000 C CNN
 F 1 "Tape/FX" H 2150 2250 50  0000 C CNN
-F 2 "Cliff:CL13345" H 2200 2650 50  0001 C CNN
+F 2 "TAC:CL13345" H 2200 2650 50  0001 C CNN
 F 3 "~" H 2200 2650 50  0001 C CNN
 	1    2200 2650
@@
 F 0 "SK3" H 2150 3900 50  0000 C CNN
 F 1 "Insert" H 2150 3200 50  0000 C CNN
-F 2 "Cliff:CL13345" H 2200 3600 50  0001 C CNN
+F 2 "TAC:CL13345" H 2200 3600 50  0001 C CNN
 F 3 "~" H 2200 3600 50  0001 C CNN
 	1    2200 3600
